Commit message: Name change

File: RobotArmModel/urdf/box assembly.SLDASM.urdf (robot description, URDF)
Before this commit: robot box assembly.SLDASM, 7 links, 6 joints
Links:
- link base_link: geometry collision mesh filename=package://RobotArmModel/meshes/base_link.STL; visual mesh filename=package://RobotArmModel/meshes/base_link.STL
- link end_effector: geometry collision mesh filename=package://RobotArmModel/meshes/end_effector.STL; visual mesh filename=package://RobotArmModel/meshes/end_effector.STL
- link link_five: geometry collision mesh filename=package://RobotArmModel/meshes/link_five.STL; visual mesh filename=package://RobotArmModel/meshes/link_five.STL
- link link_four: geometry collision mesh filename=package://RobotArmModel/meshes/link_four.STL; visual mesh filename=package://RobotArmModel/meshes/link_four.STL
- link link_one: geometry collision mesh filename=package://RobotArmModel/meshes/link_one.STL; visual mesh filename=package://RobotArmModel/meshes/link_one.STL
- link link_three: geometry collision mesh filename=package://RobotArmModel/meshes/link_three.STL; visual mesh filename=package://RobotArmModel/meshes/link_three.STL
- link link_two: geometry collision mesh filename=package://RobotArmModel/meshes/link_two.STL; visual mesh filename=package://RobotArmModel/meshes/link_two.STL
